File: Hardware_Development/PCB Designs/Dark_Passenger_Power Distro/Dark_Passenger_Power Distro.kicad_pcb (KiCad board)
At the start: 2 copper layers, 106.2 x 63 mm, 39 parts, among them J1 BATT_1, J10 RaspPi_PWR, J11 USB_HUB1_PWR, J12 USB_HUB2_PWR, J13 5V CONV, J14 BATT_MEAS, J2 BATT_2, J3 BATT_COMB, J4 5V Input, J5 BATT_CUTOFF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

Commit message: PCB Design Updates
Changed lines of the file:
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@@
 	(title_block
 		(title "Dark Passenger Power Distro Traces")
-		(date "2025-03-08")
-		(rev "V1")
+		(date "2025-03-18")
+		(rev "V2")
 		(company "Ranil Ganlath")
 	)
@@
 		)
 	)
+	(gr_text "+"
+		(at 55.25 64 0)
+		(layer "F.SilkS")
+		(effects
+			(font
+				(size 1.25 1.25)
+				(thickness 0.25)
+				(bold yes)
+			)
+			(justify left bottom)
+		)
+	)
 	(gr_text "Tonight's the night"
 		(at 85 63.5 0)
@@
 	)
 	(gr_text "-"
+		(at 60.5 64.5 0)
+		(layer "F.SilkS")
+		(effects
+			(font
+				(size 1.25 1.25)
+				(thickness 0.25)
+				(bold yes)
+			)
+			(justify left bottom)
+		)
+	)
+	(gr_text "-"
 		(at 42 58.75 270)
 		(layer "F.SilkS")
@@
 		)
 	)
+	(gr_text "-"
+		(at 60.5 63.25 180)
+		(layer "B.SilkS")
+		(effects
+			(font
+				(size 1.25 1.25)
+				(thickness 0.25)
+				(bold yes)
+			)
+			(justify left bottom mirror)
+		)
+	)
 	(gr_text "G"
 		(at 58 273.8 0)
@@
 		)
 	)
+	(gr_text "+"
+		(at 55.25 62.84 180)
+		(layer "B.SilkS")
+		(effects
+			(font
+				(size 1.25 1.25)
+				(thickness 0.25)
+				(bold yes)
+			)
+			(justify left bottom mirror)
+		)
+	)
