File: Hardware_Development/PCB Designs/Dark_Passenger_Power Distro/Dark_Passenger_Power Distro.kicad_sch (KiCad schematic)
At the start: 35 parts, among them J1 BATT_1, J10 RaspPi_PWR, J11 USB_HUB1_PWR, J12 USB_HUB2_PWR, J13 5V CONV, J14 BATT_MEAS, J2 BATT_2, J3 BATT_COMB, J4 5V Input, J5 BATT_CUTOFF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

Commit message: PCB Design Updates
Parts:
- R5: value 200ohm -> 1k
- R6: value 10kohm -> 5.6kohm
- R7: value 1.571kohm -> 1kohm
Other:
- note added: "21V = 3.2V 20V = 3.0V 19V = 2.9V 18V = 2.7V 17V = 2.6V 16V = 2.4V 15V = 2.2V"
- note added: "Fixes needed for Rev V2. Fix + and - on Terminal Blocks to match the actual components."
- note removed: "FIX RES VALUE"
Changed lines of the file:
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@@
 	(title_block
 		(title "Dark Passenger Power Distro Schematic")
-		(date "2025-03-08")
-		(rev "V1")
+		(date "2025-03-18")
+		(rev "V2")
 		(comment 1 "Email: ranil.ganlath@gmail.com")
 		(comment 2 "Author: Ranil Ganlath")
@@
 	(rectangle
 		(start 85.09 31.75)
-		(end 198.12 73.66)
+		(end 209.55 73.66)
 		(stroke
 			(width 0)
@@
 		)
 	)
+	(text "Fixes needed for Rev V2.\nFix + and - on Terminal Blocks to match the actual components."
+		(exclude_from_sim no)
+		(at 132.334 27.94 0)
+		(effects
+			(font
+				(size 5 5)
+				(italic yes)
+			)
+			(justify left bottom)
+		)
+	)
 	(text "20VDC Distribution"
 		(exclude_from_sim no)
@@
 		)
 	)
-	(text "FIX RES VALUE"
+	(text "21V = 3.2V\n20V = 3.0V\n19V = 2.9V\n18V = 2.7V\n17V = 2.6V\n16V = 2.4V\n15V = 2.2V"
 		(exclude_from_sim no)
-		(at 143.51 49.53 0)
+		(at 195.072 49.53 0)
 		(effects
 			(font
 				(size 1.27 1.27)
+				(italic yes)
 			)
 			(justify left bottom)
@@
 	(text "Voltage Divider to give 3.3V Battery Life"
 		(exclude_from_sim no)
-		(at 157.48 62.23 0)
+		(at 163.068 64.262 0)
 		(effects
 			(font
@@
 		(fields_autoplaced yes)
 		(property "Reference" "R7"
-			(at 165.1 53.975 0)
+			(at 165.1 53.3399 0)
 			(effects
 				(font
@@
 			)
 		)
-		(property "Value" "1.571kohm"
-			(at 165.1 56.515 0)
+		(property "Value" "1kohm"
+			(at 165.1 55.8799 0)
 			(effects
 				(font
@@
 		(fields_autoplaced yes)
 		(property "Reference" "R5"
-			(at 143.51 44.45 0)
+			(at 143.51 44.4499 0)
 			(effects
 				(font
@@
 			)
 		)
-		(property "Value" "200ohm"
-			(at 143.51 46.99 0)
+		(property "Value" "1k"
+			(at 143.51 46.9899 0)
 			(effects
 				(font
@@
 		(fields_autoplaced yes)
 		(property "Reference" "R6"
-			(at 165.1 43.815 0)
+			(at 165.1 43.1799 0)
 			(effects
 				(font
@@
 			)
 		)
-		(property "Value" "10kohm"
-			(at 165.1 46.355 0)
+		(property "Value" "5.6kohm"
+			(at 165.1 45.7199 0)
 			(effects
 				(font
