File: Hardware_Development/PCB Designs/Dark_Passenger_Turret_MCU/Dark_Passenger_Turret_MCU.kicad_pcb (KiCad board)
At the start: 2 copper layers, 119.4 x 61.4 mm, 39 parts, among them J1 Conn_01x22, J10 SPARE I2C, J11 IMU, J12 NEMA17 Stepper 1 ALT, J13 NEMA17 Stepper 2 ALT, J14 MS1 Jumper1, J15 MS1 Jumper2, J16 RESET, J17 NEMA17 Stepper 1, J18 NEMA17 Stepper 2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

Commit message: Updates to code based on new pinouts from PCBs
Parts:
- J10, J11: footprint Connector_PinSocket_2.54mm:PinSocket_1x04_P2.54mm_Vertical -> GanlathLib:BlankPin_1x04_P2.54mm
- J16: footprint Connector_PinSocket_2.54mm:PinSocket_1x02_P2.54mm_Vertical -> GanlathLib:BlankPin_1x02_P2.54mm
- J17, J18: footprint Connector_PinSocket_2.54mm:PinSocket_1x04_P2.54mm_Vertical -> Connector_PinHeader_2.54mm:PinHeader_1x04_P2.54mm_Vertical
