File: Hardware_Development/PCB Designs/Dark_Passenger_Turret_MCU/Dark_Passenger_Turret_MCU.kicad_sch (KiCad schematic)
At the start: 37 parts, among them J1 Conn_01x22, J10 SPARE I2C, J11 IMU, J12 NEMA17 Stepper 1 ALT, J13 NEMA17 Stepper 2 ALT, J14 MS1 Jumper1, J15 MS1 Jumper2, J16 RESET, J17 NEMA17 Stepper 1, J18 NEMA17 Stepper 2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

Commit message: Updates to code based on new pinouts from PCBs
Parts:
- C1: value C_Polarized -> 100uF
- R1: value 1k -> 300ohm
- R2: value 1k -> 130ohm
Other:
- moved on the sheet: D1, D2, D3, R1, R2, R3
