Commit message: Implemented GazeboSim

File: ROS2/dp_ws/src/dexter/description/robot_core.xacro (robot description, xacro)
@@ -46,4 +46,6 @@
     <xacro:property name="roomba_wheel_weight" value="0.1" />
     <xacro:property name="caster_wheel_radius" value="0.024" />
+    <xacro:property name="caster_wheel_weight" value="0.026" />
+    <xacro:property name="caster_wheel_center_offset" value="0.14" />
     <xacro:property name="roomba_chassis_radius" value="0.17145" />
     <xacro:property name="roomba_chassis_height" value="0.075" />
@@ -129,5 +131,5 @@
         <parent link="roomba_chassis"/>
         <child link="caster_wheel"/>
-        <origin xyz="0.14 0 ${caster_wheel_radius - roomba_wheel_height_offset}"/>
+        <origin xyz="${caster_wheel_center_offset} 0 ${caster_wheel_radius - roomba_wheel_height_offset}"/>
     </joint>
     <link name="caster_wheel">
@@ -143,5 +145,5 @@
             </geometry>
         </collision>
-        <xacro:inertial_sphere mass="0.1" radius="${caster_wheel_radius}">
+        <xacro:inertial_sphere mass="${caster_wheel_weight}" radius="${caster_wheel_radius}">
             <origin xyz="0 0 0" rpy= "0 0 0"/>
         </xacro:inertial_sphere>

Commit message: Modified control plugins to interface with Gazebo Harmonic

File: ROS2/dp_ws/src/dexter/description/robot_core.xacro (robot description, xacro)
@@ -81,4 +81,7 @@
         </xacro:inertial_cylinder>
     </link>
+    <gazebo reference="roomba_chassis">
+        <material>Gazebo/White</material>
+    </gazebo>
 <!-- LEFT WHEEL Link -->
     <joint name="left_wheel_joint" type="continuous">
@@ -104,4 +107,7 @@
         </xacro:inertial_cylinder>
     </link>
+    <gazebo reference="left_wheel">
+        <material>Gazebo/Blue</material>
+    </gazebo>
 <!-- RIGHT WHEEL Link -->
     <joint name="right_wheel_joint" type="continuous">
@@ -127,4 +133,7 @@
         </xacro:inertial_cylinder>
     </link>
+    <gazebo reference="right_wheel">
+        <material>Gazebo/Red</material>
+    </gazebo>
 <!-- CASTER WHEEL Link -->
     <joint name="caster_wheel_joint" type="fixed">
@@ -149,4 +158,9 @@
         </xacro:inertial_sphere>
     </link>
+    <gazebo reference="caster_wheel">
+        <material>Gazebo/Blue</material>
+        <mu1 value="0.001"/>
+        <mu2 value="0.001"/>
+    </gazebo>
  <!-- Payload Chassis Link -->
     <joint name="payload_chassis_joint" type="fixed">
@@ -173,3 +187,6 @@
         </xacro:inertial_box>
     </link>
+    <gazebo reference="payload_chassis">
+        <material>Gazebo/Green</material>
+    </gazebo>
 </robot>
