Commit message: Removed collision physics for Lidar since internal to box.

File: ROS2/dp_ws/src/dexter/description/lidar.xacro (robot description, xacro)
@@ -20,12 +20,4 @@
             <material name="black"/>
         </visual>
-        <collision>
-            <geometry>
-                <cylinder radius="0.05" length="0.02"/>
-            </geometry>
-        </collision>
-        <xacro:inertial_cylinder mass="0.1" length="0.02" radius="0.035">
-            <origin xyz="0 0 0" rpy="0 0 0"/>
-        </xacro:inertial_cylinder>
     </link>
     <gazebo reference="laser_frame">
@@ -33,5 +25,5 @@
         <sensor name="laser" type="gpu_lidar">
             <pose> 0 0 0 0 0 0 </pose>
-            <visualize>false</visualize>
+            <visualize>true</visualize>
             <update_rate>10</update_rate>
             <lidar>
