Commit message: Passing launch parameters to rsp.launch

File: ROS2/dp_ws/src/dexter/description/robot.urdf.xacro (robot description, xacro)
@@ -1,7 +1,13 @@
 <?xml version="1.0"?>
 <robot xmlns:xacro="http://www.ros.org/wiki/xacro"  name="robot">
+    <xacro:arg name="use_ros2_control" default="true"/>
+    <xacro:arg name="sim_mode" default="false"/>
     <xacro:include filename="robot_core.xacro" />
-    <!-- <xacro:include filename="gazebo_control.xacro"/> -->
-    <xacro:include filename="ros2_control.xacro"/>
+    <xacro:if value="$(arg use_ros2_control)">
+        <xacro:include filename="ros2_control.xacro" />
+    </xacro:if>
+    <xacro:unless value="$(arg use_ros2_control)">
+        <xacro:include filename="gazebo_control.xacro" />
+    </xacro:unless>
     <xacro:include filename="lidar.xacro" />
     <!-- <xacro:include filename="camera.xacro" /> -->

File: ROS2/dp_ws/src/dexter/description/robot_core.xacro (robot description, xacro)
@@ -100,5 +100,5 @@
         <collision>
             <geometry>
-                <cylinder radius="${roomba_wheel_radius}" length="${roomba_wheel_thickness}"/>
+                <sphere radius="${roomba_wheel_radius}"/>
             </geometry>
         </collision>
@@ -126,5 +126,5 @@
         <collision>
             <geometry>
-                <cylinder radius="${roomba_wheel_radius}" length="${roomba_wheel_thickness}"/>
+                <sphere radius="${roomba_wheel_radius}"/>
             </geometry>
         </collision>
